Commit message: implemented joint state publisher

File: description/jetbot.urdf (robot description, URDF)
Before this commit: robot JetBot, 4 links, 3 joints
Joints:
- joint JetBot__left_wheel_hinge: limit lower=0 upper=0 effort=0 velocity=0 -> effort=1 velocity=1; type fixed -> continuous
- joint JetBot__right_wheel_hinge: limit lower=0 upper=0 effort=0 velocity=0 -> effort=1 velocity=1; type fixed -> continuous
