Commit message: got robot state publisher working

File: description/urdf/jetbot.urdf (robot description, URDF)
Before this commit: robot JetBot, 4 links, 3 joints
Links:
- added link base_link
- added link odom
Joints:
- added joint base_link_joint: type fixed, parent base_link, child JetBot__chassis, origin xyz=0 0 0 rpy=0 0 0
- added joint odom_joint: type fixed, parent odom, child base_link, origin xyz=0 0 0 rpy=0 0 0
- joint JetBot__right_wheel_hinge: origin xyz=0.03   -0.05125  0.03 rpy=0      0      -1.57079 -> xyz=0.03   -0.05125  0.03 rpy=0      0      1.57079
