Commit message: added imu stl

File: jetbot_description/urdf/jetbot.urdf (robot description, URDF)
Before this commit: robot JetBot, 6 links, 5 joints
Links:
- added link JetBot__imu_link; visual mesh filename=package://description/meshes/MPU-6050.stl scale=0.001 0.001 0.001
Joints:
- added joint imu_link: type fixed, parent JetBot__chassis, child JetBot__imu_link, origin xyz=0 0 0 rpy=0 0 0, axis 0 0 0

Commit message: saved new imu rotation params and updated the urdf

File: jetbot_description/urdf/jetbot.urdf (robot description, URDF)
Before this commit: robot JetBot, 7 links, 6 joints
Joints:
- removed joint imu_link
- added joint JetBot__imu_joint: type fixed, parent JetBot__chassis, child JetBot__imu_link, origin xyz=-0.055 0.051215 0.03 rpy=125.311 87.2866 -123.066, axis 0 0 0

Commit message: Fixed urdf file which used outdated pkg names

File: jetbot_description/urdf/jetbot.urdf (robot description, URDF)
Before this commit: robot JetBot, 6 links, 5 joints
Links:
- link JetBot__chassis: geometry collision mesh filename=package://jetbot_description/meshes/JetBot-v3-Chassis.dae scale=0.001 0.001 0.001; visual mesh filename=package://jetbot_description/meshes/JetBot-v3-Chassis.dae scale=0.001 0.001 0.001
- link JetBot__left_wheel: geometry collision mesh filename=package://jetbot_description/meshes/JetBot-v3-Wheel.stl scale=0.001 0.001 0.001; visual mesh filename=package://jetbot_description/meshes/JetBot-v3-Wheel.stl scale=0.001 0.001 0.001
- link JetBot__right_wheel: geometry collision mesh filename=package://jetbot_description/meshes/JetBot-v3-Wheel.stl scale=0.001 0.001 0.001; visual mesh filename=package://jetbot_description/meshes/JetBot-v3-Wheel.stl scale=0.001 0.001 0.001

Commit message: fixed sign on acceleration reading

File: jetbot_description/urdf/jetbot.urdf (robot description, URDF)
Before this commit: robot JetBot, 7 links, 6 joints
Links:
- link JetBot__imu_link: mass None -> 0; geometry collision mesh filename=package://jetbot_description/meshes/MPU-6050.stl scale=0.023 0.023 0.023; visual mesh filename=package://jetbot_description/meshes/MPU-6050.stl scale=0.023 0.023 0.023
Joints:
- joint JetBot__imu_joint: origin xyz=-0.055 0.051215 0.03 rpy=125.311 87.2866 -123.066 -> xyz=-0.065 0.035 0.017 rpy=0 1.57079 0

Commit message: corrected pose of imu in urdf

File: jetbot_description/urdf/jetbot.urdf (robot description, URDF)
Before this commit: robot JetBot, 7 links, 6 joints
Joints:
- joint JetBot__imu_joint: origin xyz=-0.065 0.035 0.017 rpy=0 1.57079 0 -> xyz=-0.065 0.035 0.017 rpy=1.57079 0 1.57079

Commit message: Fixed wheel seperation in urdf

File: jetbot_description/urdf/jetbot.urdf (robot description, URDF)
Before this commit: robot JetBot, 6 links, 5 joints
Joints:
- joint JetBot__left_wheel_hinge: origin xyz=0.03    0.05125 0.03 rpy=0      0      1.57079 -> xyz=0.03    0.0475 0.03 rpy=0      0      1.57079
- joint JetBot__right_wheel_hinge: origin xyz=0.03   -0.05125  0.03 rpy=0      0      1.57079 -> xyz=0.03   -0.056  0.03 rpy=0      0      1.57079

Commit message: created and ran transformer pkg locally

File: jetbot_description/urdf/jetbot.urdf (robot description, URDF)
Before this commit: robot JetBot, 7 links, 6 joints
Links:
- link JetBot__imu_link: mass 0 -> None; geometry visual mesh filename=package://jetbot_description/meshes/MPU-6050.stl scale=0.023 0.023 0.023
Joints:
- joint JetBot__imu_joint: origin xyz=-0.065 0.035 0.017 rpy=1.57079 0 1.57079 -> xyz=-0.065 0.035 0.017 rpy=1.57079 -1.57079 0

Commit message: write mpu 6050 driver (#12)
added imu pkg + transformer pkg

File: jetbot_description/urdf/jetbot.urdf (robot description, URDF)
Before this commit: robot JetBot, 6 links, 5 joints
Links:
- added link JetBot__imu_link; visual mesh filename=package://jetbot_description/meshes/MPU-6050.stl scale=0.023 0.023 0.023
Joints:
- added joint JetBot__imu_joint: type fixed, parent JetBot__chassis, child JetBot__imu_link, origin xyz=-0.065 0.035 0.017 rpy=1.57079 -1.57079 0, axis 0 0 0
